File: hardware/jlink_to_tag/rev_e/jlink_to_tag.sch (EAGLE design)
At the start: 14 parts, among them J2 JLINK_6PIN_TAG-CON, U1 LT1763CS8-3.3

Commit message: update part numbers
Parts:
- R2, R3: device passives:RESISTOR0402_RES -> passives:RESISTOR0603_RES
- S2, S3: DIGIKEY (none) -> 2223-SLW-883935-2A-D-ND; MPN (none) -> SLW-883935-2A-D
Changed lines of the file:
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@@
 <part name="R1" library="SparkFun-Passives" deviceset="RESISTOR" device="0603-RES" value="470"/>
 <part name="S1" library="switches" deviceset="EVQP2" device=""/>
-<part name="S2" library="switches" deviceset="TE_SSA12/SPDT" device=""/>
+<part name="S2" library="switches" deviceset="TE_SSA12/SPDT" device="">
+<attribute name="DIGIKEY" value="2223-SLW-883935-2A-D-ND"/>
+<attribute name="MPN" value="SLW-883935-2A-D"/>
+</part>
 <part name="GND3" library="SparkFun-Aesthetics" deviceset="GND" device=""/>
-<part name="S3" library="switches" deviceset="TE_SSA12/SPDT" device=""/>
+<part name="S3" library="switches" deviceset="TE_SSA12/SPDT" device="">
+<attribute name="DIGIKEY" value="2223-SLW-883935-2A-D-ND"/>
+<attribute name="MPN" value="SLW-883935-2A-D"/>
+</part>
 <part name="S4" library="switches" deviceset="OS103011MS8QP1" device=""/>
-<part name="R2" library="passives" deviceset="RESISTOR" device="0402_RES" value="10k"/>
-<part name="R3" library="passives" deviceset="RESISTOR" device="0402_RES" value="20k"/>
+<part name="R2" library="passives" deviceset="RESISTOR" device="0603_RES" value="10k"/>
+<part name="R3" library="passives" deviceset="RESISTOR" device="0603_RES" value="20k"/>
 <part name="GND8" library="SparkFun-Aesthetics" deviceset="GND" device=""/>
 </parts>
@@
 <attribute name="NAME" x="99.06" y="76.2" size="1.27" layer="95"/>
 <attribute name="VALUE" x="99.06" y="73.66" size="1.27" layer="96"/>
+<attribute name="MPN" x="101.6" y="83.82" size="1.778" layer="96" display="off"/>
 </instance>
 <instance part="GND3" gate="1" x="45.72" y="76.2" smashed="yes">
@@
 <attribute name="NAME" x="101.6" y="33.02" size="1.27" layer="95"/>
 <attribute name="VALUE" x="101.6" y="30.48" size="1.27" layer="96"/>
+<attribute name="MPN" x="104.14" y="40.64" size="1.778" layer="96" display="off"/>
 </instance>
 <instance part="S4" gate="G$1" x="101.6" y="114.3" smashed="yes">

Commit message: add BOM and final changes
Parts:
- D1: DIGIKEY (none) -> 160-1827-1-ND
- R1: DIGIKEY (none) -> P470DBCT-ND
- R2: DIGIKEY (none) -> RMCF0603FT10K0CT-ND
- R3: DIGIKEY (none) -> P20.0KHCT-ND
Changed lines of the file:
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@@
 <attribute name="DIGIKEY" value="S9172-ND"/>
 </part>
-<part name="D1" library="SparkFun-LED" deviceset="LED-BLUE" device="0603" value="BLUE"/>
+<part name="D1" library="SparkFun-LED" deviceset="LED-BLUE" device="0603" value="BLUE">
+<attribute name="DIGIKEY" value="160-1827-1-ND"/>
+</part>
 <part name="GND1" library="SparkFun-Aesthetics" deviceset="GND" device=""/>
 <part name="GND2" library="SparkFun-Aesthetics" deviceset="GND" device=""/>
@@
 </part>
 <part name="FRAME1" library="frames" deviceset="LETTER_L" device=""/>
-<part name="R1" library="SparkFun-Passives" deviceset="RESISTOR" device="0603-RES" value="470"/>
+<part name="R1" library="SparkFun-Passives" deviceset="RESISTOR" device="0603-RES" value="470">
+<attribute name="DIGIKEY" value="P470DBCT-ND"/>
+</part>
 <part name="S1" library="switches" deviceset="EVQP2" device=""/>
 <part name="S2" library="switches" deviceset="TE_SSA12/SPDT" device="">
@@
 </part>
 <part name="S4" library="switches" deviceset="OS103011MS8QP1" device=""/>
-<part name="R2" library="passives" deviceset="RESISTOR" device="0603_RES" value="10k"/>
-<part name="R3" library="passives" deviceset="RESISTOR" device="0603_RES" value="20k"/>
+<part name="R2" library="passives" deviceset="RESISTOR" device="0603_RES" value="10k">
+<attribute name="DIGIKEY" value="RMCF0603FT10K0CT-ND"/>
+</part>
+<part name="R3" library="passives" deviceset="RESISTOR" device="0603_RES" value="20k">
+<attribute name="DIGIKEY" value="P20.0KHCT-ND"/>
+</part>
 <part name="GND8" library="SparkFun-Aesthetics" deviceset="GND" device=""/>
 </parts>
@@
 <attribute name="NAME" x="191.516" y="132.588" size="1.778" layer="95" rot="R90"/>
 <attribute name="VALUE" x="193.675" y="132.588" size="1.778" layer="96" rot="R90"/>
+<attribute name="DIGIKEY" x="187.96" y="137.16" size="1.778" layer="96" display="off"/>
 </instance>
 <instance part="GND1" gate="1" x="22.86" y="119.38" smashed="yes">
@@
 <attribute name="NAME" x="189.4586" y="151.13" size="1.778" layer="95" rot="R270"/>
 <attribute name="VALUE" x="184.658" y="151.13" size="1.778" layer="96" rot="R270"/>
+<attribute name="DIGIKEY" x="187.96" y="147.32" size="1.778" layer="96" rot="R270" display="off"/>
 </instance>
 <instance part="S1" gate="G$1" x="35.56" y="83.82" smashed="yes">
@@
 <attribute name="NAME" x="128.0414" y="85.09" size="1.778" layer="95" rot="R90"/>
 <attribute name="VALUE" x="132.842" y="85.09" size="1.778" layer="96" rot="R90"/>
+<attribute name="DIGIKEY" x="129.54" y="88.9" size="1.778" layer="96" rot="R90" display="off"/>
 </instance>
 <instance part="R3" gate="G$1" x="129.54" y="76.2" smashed="yes" rot="R90">
 <attribute name="NAME" x="128.0414" y="72.39" size="1.778" layer="95" rot="R90"/>
 <attribute name="VALUE" x="132.842" y="72.39" size="1.778" layer="96" rot="R90"/>
+<attribute name="DIGIKEY" x="129.54" y="76.2" size="1.778" layer="96" rot="R90" display="off"/>
 </instance>
 <instance part="GND8" gate="1" x="129.54" y="66.04" smashed="yes">
